File: corbit.kicad_sch (KiCad schematic)
At the start: 45 parts, among them J1 Conn_01x02, SW1 SW_Push, SW10 SW_Push, SW11 SW_Push, SW12 SW_Push, SW13 SW_Push, SW14 SW_Push, SW15 SW_Push, SW16 SW_Push, SW17 SW_Push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

Commit message: change matrix and add rotary encoder in scketch
Parts:
- removed D21: D, symbol Device:D
- removed SW21: SW_Push, symbol Switch:SW_Push
- added SW21: RotaryEncoder, symbol Device:RotaryEncoder
Connections:
- net Col0: now also SW11.1, SW16.1, SW6.1, U1.5 (P0.04_A4_D4_SDA); no longer SW15.1, SW8.1, U1.4 (P0.29_A3_D3)
- net Col1: now also SW12.1, SW17.1, SW7.1, U1.6 (P0.05_A5_D5_SCL); no longer SW16.1, SW9.1, U1.5 (P0.04_A4_D4_SDA)
- net Col2: now also SW13.1, SW18.1, SW8.1, U1.7 (P1.11_D6_TX); no longer SW10.1, SW17.1, U1.6 (P0.05_A5_D5_SCL)
- net Col3: now also SW14.1, SW19.1, SW9.1, U1.8 (P1.12_D7_RX); no longer SW11.1, SW18.1, U1.7 (P1.11_D6_TX)
- net Col4: now also SW10.1, SW15.1, SW20.1, U1.9 (P1.13_D8_SCK); no longer SW12.1, SW19.1, U1.10 (P1.14_D9_MISO)
- net GND: now also SW21.C
- net Row0: no longer D6.1 (K), D7.1 (K)
- net Row1: now also D6.1 (K), D7.1 (K); no longer D11.1 (K), D12.1 (K), D13.1 (K), D14.1 (K)
- net Row2: now also D11.1 (K), D12.1 (K), D13.1 (K), D14.1 (K); no longer D16.1 (K), D17.1 (K), D18.1 (K), D19.1 (K), D20.1 (K)
- net RotA: now reaches U1.11 (P1.15_D10_MOSI)
- net RotA: now also SW21.A
- removed net Col5: SW13.1, SW20.1, SW6.1, U1.9 (P1.13_D8_SCK)
- removed net Col6: SW14.1, SW7.1, U1.8 (P1.12_D7_RX)
- new net RotB: SW21.B, U1.10 (P1.14_D9_MISO)
- new net Row3: D16.1 (K), D17.1 (K), D18.1 (K), D19.1 (K), D20.1 (K), U1.4 (P0.29_A3_D3)
- no-connect marks 16 -> 15
Other:
- moved on the sheet: D10, D11, D12, D13, D14, D15, D16, D17, D18, D19, D20, D6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

Commit message: footprints
Parts:
- D1, D10, D11, D12, D13, D14, D15, D16, D17, D18, D19, D2, D20, D3, D4, D5, D6, D8, D9: footprint (none) -> Diode_SMD:D_SOD-123
- Deee1: renamed from D7; footprint (none) -> Diode_SMD:D_SOD-123
- J1: footprint (none) -> Connector_JST:JST_PH_S2B-PH-K_1x02_P2.00mm_Horizontal
- SW1, SW10, SW11, SW12, SW13, SW14, SW15, SW16, SW17, SW18, SW19, SW2, SW20, SW3, SW4, SW5, SW6, SW7, SW8, SW9: footprint (none) -> corbit:SW_Hotswap_Kailh_Choc_V1_1.00u-NoClickHole
- SW22: footprint (none) -> Button_Switch_SMD:SW_SPDT_PCM12
- U1: footprint Seeed_Studio_XIAO_Series:XIAO-nRF52840-Plus-SMD -> corbit:XIAO_nRF52840_plus_mki; symbol SeedStudio:XIAO-nRF52840_Plus_SMD -> smkbd_Library:XIAO-nRF52840_plus_maked_by_mki
Connections:
- net GND: now also U1.15 (BATT-), U1.26 (GND); no longer U1.27 (GND), U1.33 (GND)
- net VBAT_SW: now also U1.16 (BATT+); no longer U1.32 (VBAT)
- no-connect marks 15 -> 13
Other:
- moved on the sheet: D1, D10, D11, D12, D13, D14, D15, D16, D17, D18, D19, D2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

Commit message: generated PCB
Parts:
- SW21: footprint (none) -> corbit:rotary_encoder_EC05E_Vert
Changed lines of the file:
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@@
 			)
 		)
-		(property "Footprint" ""
+		(property "Footprint" "corbit:rotary_encoder_EC05E_Vert"
 			(at 125.73 103.886 0)
 			(hide yes)

Commit message: edit pcb
Parts:
- renumbered Deee1 to D7
Changed lines of the file:
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@@
 		(dnp no)
 		(fields_autoplaced yes)
-		(property "Reference" "Deee1"
+		(property "Reference" "D7"
 			(at 59.69 124.4599 90)
 			(show_name no)
@@
 			(project "corbit"
 				(path "/46fee64b-d8d5-4529-99df-0fd09c2b7c9b"
-					(reference "Deee1")
+					(reference "D7")
 					(unit 1)
 				)
