File: corbit.kicad_pcb (KiCad board)
At the start: 2 copper layers, 6.1 x 13.9 mm, 44 parts, among them J1 Conn_01x02, SW1 SW_Push, SW10 SW_Push, SW11 SW_Push, SW12 SW_Push, SW13 SW_Push, SW14 SW_Push, SW15 SW_Push, SW16 SW_Push, SW17 SW_Push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

Commit message: edit pcb
Parts:
- moved SW17 111.1 mm to (61.0, 113.0), turned to 180 degrees
- moved D5 104.0 mm to (160.0, 73.0), turned to 90 degrees
- moved D4 89.9 mm to (142.0, 72.0), turned to 90 degrees
- moved U1 88.4 mm to (172.1, 71.0)
- moved SW16 87.4 mm to (61.0, 96.0), turned to 180 degrees
- moved D10 86.6 mm to (160.0, 90.0), turned to 90 degrees
- moved D3 78.3 mm to (124.0, 70.0), turned to 90 degrees
- moved D20 75.9 mm to (176.0, 127.0), turned to 150 degrees
- moved D15 72.7 mm to (160.0, 107.0), turned to 90 degrees
- moved D9 71.1 mm to (142.0, 89.0), turned to 90 degrees
- moved D2 69.5 mm to (106.0, 68.0), turned to 90 degrees
- moved SW22 67.9 mm to (180.7, 99.5), turned to 90 degrees
- moved SW4 63.2 mm to (133.0, 75.0), turned to 180 degrees
- moved D19 60.8 mm to (162.0, 133.0), turned to 75 degrees
- moved SW21 59.3 mm to (191.0, 131.0), turned to -30 degrees
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- renumbered Deee1 to D7
Other:
- board size 6.1 x 13.9 mm -> 147 x 94 mm

Commit message: edit outline
Parts:
- moved J1 4.12 mm to (178.4, 93.0)
- moved SW22 4.00 mm to (180.7, 103.5)
- moved U1 4.00 mm to (172.1, 75.0)
Other:
- outline, holes or cut-outs redrawn
Changed lines of the file:
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@@
 	(footprint "Button_Switch_SMD:SW_SPDT_PCM12"
 		(layer "F.Cu")
-		(at 180.67 99.5 90)
+		(at 180.67 103.5 90)
 		(descr "Ultraminiature Surface Mount Slide Switch, right-angle, https://www.ckswitches.com/media/1424/pcm.pdf")
 		(property "Reference" "SW22"
@@
 		(fp_line
 			(start -0.35 0.000001)
-			(end -0.35 0.550001)
+			(end -0.35 0.550002)
 			(stroke
 				(width 0.1)
@@
 	(footprint "Connector_JST:JST_PH_S2B-PH-K_1x02_P2.00mm_Horizontal"
 		(layer "F.Cu")
-		(at 177.45 89 -90)
+		(at 178.45 93 -90)
 		(descr "JST PH series connector, S2B-PH-K (http://www.jst-mfg.com/product/pdf/eng/ePH.pdf)")
 		(tags "connector JST PH horizontal")
@@
 	(footprint "corbit:XIAO_nRF52840_plus_mki"
 		(layer "F.Cu")
-		(at 172.0635 70.985)
+		(at 172.0635 74.985)
 		(property "Reference" "U1"
 			(at -0.02 0.06 0)
@@
 	)
 	(gr_line
+		(start 124 62)
+		(end 88 62)
+		(stroke
+			(width 0.05)
+			(type default)
+		)
+		(layer "Edge.Cuts")
+	)
+	(gr_line
+		(start 151 66)
+		(end 124 62)
+		(stroke
+			(width 0.05)
+			(type default)
+		)
+		(layer "Edge.Cuts")
+	)
+	(gr_line
 		(start 171.599938 148.342822)
 		(end 122.322829 137.939224)
@@
 	)
 	(gr_line
-		(start 179 62)
-		(end 88 62)
+		(start 179 66)
+		(end 151 66)
 		(stroke
 			(width 0.05)
@@
 	)
 	(gr_arc
-		(start 179 62)
-		(mid 181.828427 63.171573)
-		(end 183 66)
+		(start 179 66)
+		(mid 181.828427 67.171573)
+		(end 183 70)
 		(stroke
 			(width 0.05)
@@
 	(gr_line
 		(start 183 127)
-		(end 183 66)
+		(end 183 70)
 		(stroke
 			(width 0.05)
