File: corbit.kicad_pcb (KiCad board)
At the start: 2 copper layers, 147 x 94 mm, 44 parts, among them J1 Conn_01x02, SW1 SW_Push, SW10 SW_Push, SW11 SW_Push, SW12 SW_Push, SW13 SW_Push, SW14 SW_Push, SW15 SW_Push, SW16 SW_Push, SW17 SW_Push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

Commit message: dit
Parts:
- moved D20 1.00 mm to (176.0, 127.0), turned to -30 degrees
- moved SW20 0.34 mm to (173.0, 136.0)
Other:
- board size 147 x 94 mm -> 144 x 92 mm
Changed lines of the file:
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@@
 	(footprint "corbit:SW_Hotswap_Kailh_Choc_V1_1.00u-NoClickHole"
 		(layer "F.Cu")
-		(at 172.75 136.23686 -120)
+		(at 173 136 -120)
 		(descr "Kailh keyswitch Hotswap Socket with 1.00u keycap")
 		(tags "Kailh Keyboard Choc V1 keyswitch Keyswitch Switch Hotswap Socket Cutout 1.00u")
@@
 		(fp_line
 			(start -0.35 -0.000001)
-			(end -0.35 0.550001)
+			(end -0.35 0.550002)
 			(stroke
 				(width 0.1)
@@
 	(footprint "Diode_SMD:D_SOD-123"
 		(layer "B.Cu")
-		(at 176 128 150)
+		(at 176 127 -30)
 		(descr "SOD-123")
 		(tags "SOD-123")
@@
 		)
 		(property "Datasheet" ""
-			(at 0 0 330)
+			(at 0 0 150)
 			(unlocked yes)
 			(layer "B.Fab")
@@
 		)
 		(property "Description" "Diode"
-			(at 0 0 330)
+			(at 0 0 150)
 			(unlocked yes)
 			(layer "B.Fab")
@@
 		)
 		(property "Sim.Device" "D"
-			(at 0 0 330)
+			(at 0 0 150)
 			(unlocked yes)
 			(layer "B.Fab")
@@
 		)
 		(property "Sim.Pins" "1=K 2=A"
-			(at 0 0 330)
+			(at 0 0 150)
 			(unlocked yes)
 			(layer "B.Fab")
@@
 		(duplicate_pad_numbers_are_jumpers no)
 		(fp_line
-			(start -2.36 -1)
-			(end 1.65 -1)
+			(start -2.36 1)
+			(end -2.36 -1)
 			(stroke
 				(width 0.12)
@@
 		)
 		(fp_line
-			(start -2.36 1)
-			(end -2.36 -1)
+			(start -2.36 -1)
+			(end 1.65 -1)
 			(stroke
 				(width 0.12)
@@
 		)
 		(fp_line
-			(start 2.35 -1.15)
+			(start -2.35 1.15)
 			(end -2.35 -1.15)
 			(stroke
@@
 		)
 		(fp_line
-			(start 2.35 1.15)
-			(end 2.35 -1.15)
+			(start -2.35 1.15)
+			(end 2.35 1.15)
 			(stroke
 				(width 0.05)
@@
 		)
 		(fp_line
-			(start -2.35 1.15)
-			(end 2.35 1.15)
+			(start 2.35 1.15)
+			(end 2.35 -1.15)
 			(stroke
 				(width 0.05)
@@
 		)
 		(fp_line
-			(start -2.35 1.15)
+			(start 2.35 -1.15)
 			(end -2.35 -1.15)
 			(stroke
@@
 		)
 		(fp_line
-			(start 1.4 -0.9)
-			(end -1.4 -0.9)
+			(start -1.4 0.9)
+			(end 1.4 0.9)
 			(stroke
 				(width 0.1)
@@
 		)
 		(fp_line
-			(start 1.4 0.9)
-			(end 1.4 -0.9)
+			(start -1.4 -0.9)
+			(end -1.4 0.9)
 			(stroke
 				(width 0.1)
@@
 		)
 		(fp_line
-			(start 0.25 -0.4)
+			(start -0.75 0)
 			(end -0.35 0)
 			(stroke
@@
 		)
 		(fp_line
-			(start 0.25 0)
-			(end 0.75 0)
+			(start -0.35 0)
+			(end -0.35 0.55)
 			(stroke
 				(width 0.1)
@@
 		)
 		(fp_line
-			(start 0.25 0.4)
-			(end 0.25 -0.4)
+			(start -0.35 0)
+			(end -0.35 -0.55)
 			(stroke
 				(width 0.1)
@@
 		)
 		(fp_line
-			(start -0.35 0)
-			(end -0.35 -0.55)
+			(start 0.25 0.4)
+			(end 0.25 -0.4)
 			(stroke
 				(width 0.1)
@@
 		)
 		(fp_line
-			(start -0.35 0)
-			(end -0.35 0.55)
+			(start 0.25 0)
+			(end 0.75 0)
 			(stroke
 				(width 0.1)
@@
 		)
 		(fp_line
-			(start -0.75 0)
+			(start 0.25 -0.4)
 			(end -0.35 0)
 			(stroke
@@
 		)
 		(fp_line
-			(start -1.4 -0.9)
-			(end -1.4 0.9)
+			(start 1.4 0.9)
+			(end 1.4 -0.9)
 			(stroke
 				(width 0.1)
@@
 		)
 		(fp_line
-			(start -1.4 0.9)
-			(end 1.4 0.9)
+			(start 1.4 -0.9)
+			(end -1.4 -0.9)
 			(stroke
 				(width 0.1)
@@
 		)
 		(pad "1" smd roundrect
-			(at -1.65 0 150)
+			(at -1.65 0 330)
 			(size 0.9 1.2)
 			(layers "B.Cu" "B.Mask" "B.Paste")
@@
 		)
 		(pad "2" smd roundrect
-			(at 1.65 0 150)
+			(at 1.65 0 330)
 			(size 0.9 1.2)
 			(layers "B.Cu" "B.Mask" "B.Paste")
@@
 	)
 	(gr_line
-		(start 171.599938 148.342822)
+		(start 168 146)
 		(end 122.322829 137.939224)
 		(stroke
@@
 	)
 	(gr_line
-		(start 183 127)
-		(end 183 70)
+		(start 182 154)
+		(end 168 146)
 		(stroke
 			(width 0.05)
@@
 	)
 	(gr_line
-		(start 183 127)
-		(end 197 135)
+		(start 182 154)
+		(end 194 133)
 		(stroke
 			(width 0.05)
@@
 	)
 	(gr_line
-		(start 185 156)
-		(end 171.599938 148.342822)
+		(start 183 125)
+		(end 183 70)
+		(stroke
+			(width 0.05)
+			(type default)
+		)
+		(layer "Edge.Cuts")
+	)
+	(gr_arc
+		(start 184.335899 127.496151)
+		(mid 183.354976 126.415574)
+		(end 183 125)
 		(stroke
 			(width 0.05)
@@
 	)
 	(gr_line
-		(start 185 156)
-		(end 197 135)
+		(start 184.335899 127.496151)
+		(end 194 133)
 		(stroke
 			(width 0.05)
