File: right/reel-right.kicad_sch (KiCad schematic)
At the start: 44 parts, among them J1 Conn_01x02, SW1 SW_Push, SW10 SW_Push, SW11 SW_Push, SW12 SW_Push, SW13 SW_Push, SW14 SW_Push, SW15 SW_Push, SW16 SW_Push, SW17 SW_Push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

Commit message: dit
Parts:
- removed SW21: RotaryEncoder, reel:rotary_encoder_EC05E_Vert, symbol Device:RotaryEncoder
- added J2: (no value), reel:pmw3610_connector, symbol reel:pmw3610_breakout
Connections:
- net Col1: now also U1.21 (GPIO_0.10); no longer U1.6 (P0.05_A5_D5_SCL)
- net GND: now also J2.3 (GND)
- net 3.3V: now reaches U1.12 (3V3)
- net 3.3V: now also J2.4 (Vin)
- net nCS: now reaches U1.24 (GPIO_1.05)
- net nCS: now also J2.2 (nCS)
- net RotA renamed SDIO
- net SDIO: now also J2.6 (SDIO)
- net RotB renamed MOTION
- net MOTION: now also J2.7 (MOTION)
- new net SCLK: J2.1 (SCLK), U1.6 (P0.05_A5_D5_SCL)
- no-connect marks 13 -> 11
