File: right/reel-right.kicad_sch (KiCad schematic)
At the start: 42 parts, among them J1 Conn_01x02, SW1 SW_Push, SW10 SW_Push, SW11 SW_Push, SW12 SW_Push, SW13 SW_Push, SW14 SW_Push, SW15 SW_Push, SW16 SW_Push, SW17 SW_Push, SW18 SW_Push, SW19 SW_Push, SW2 SW_Push, SW22 SW_SPDT, SW3 SW_Push, SW4 SW_Push, SW5 SW_Push, SW6 SW_Push, SW7 SW_Push, SW8 SW_Push, SW9 SW_Push

Commit message: Update ReeL KiCad libraries and board
Parts:
- U1: symbol roba:XIAO-nRF52840 -> reel:XIAO-nRF52840
Changed lines of the file:
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@@
 	)
 	(symbol
-		(lib_id "roba:XIAO-nRF52840")
+		(lib_id "reel:XIAO-nRF52840")
 		(at 24.13 22.86 0)
 		(unit 1)

Commit message: Update ReeL KiCad board files
Parts:
- D1, D10, D11, D12, D13, D14, D15, D16, D17, D18, D19, D2, D3, D4, D5, D6, D7, D8, D9: footprint Diode_SMD:D_SOD-123 -> reel:Diode_SMD
- SW1, SW10, SW11, SW12, SW13, SW14, SW15, SW16, SW17, SW18, SW19, SW2, SW3, SW4, SW5, SW6, SW7, SW8, SW9: footprint reel:SW_Hotswap_Kailh_Choc_V1_1.00u-NoClickHole -> reel:SW_Hotswap_Kailh_Choc_V1V2_1.00u
Changed lines of the file:
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@@
 	)
 	(junction
-		(at 72.39 113.03)
-		(diameter 0)
-		(color 0 0 0 0)
-	)
-	(junction
-		(at 57.15 146.05)
-		(diameter 0)
-		(color 0 0 0 0)
-	)
-	(junction
 		(at 62.23 121.92)
 		(diameter 0)
@@
 	)
 	(junction
+		(at 72.39 113.03)
+		(diameter 0)
+		(color 0 0 0 0)
+	)
+	(junction
 		(at 41.91 146.05)
 		(diameter 0)
@@
 	)
 	(junction
+		(at 57.15 146.05)
+		(diameter 0)
+		(color 0 0 0 0)
+	)
+	(junction
 		(at 41.91 113.03)
 		(diameter 0)
@@
 	(wire
 		(pts
-			(xy 72.39 113.03) (xy 87.63 113.03)
+			(xy 41.91 129.54) (xy 57.15 129.54)
 		)
 		(stroke
@@
 	(wire
 		(pts
-			(xy 41.91 129.54) (xy 57.15 129.54)
+			(xy 29.21 146.05) (xy 41.91 146.05)
 		)
 		(stroke
@@
 	(wire
 		(pts
-			(xy 29.21 146.05) (xy 41.91 146.05)
+			(xy 140.97 138.43) (xy 140.97 132.08)
 		)
 		(stroke
@@
 	(wire
 		(pts
-			(xy 140.97 138.43) (xy 140.97 132.08)
+			(xy 138.43 129.54) (xy 144.78 129.54)
 		)
 		(stroke
@@
 	(wire
 		(pts
-			(xy 138.43 129.54) (xy 144.78 129.54)
+			(xy 72.39 113.03) (xy 87.63 113.03)
 		)
 		(stroke
@@
 	(wire
 		(pts
-			(xy 57.15 146.05) (xy 72.39 146.05)
+			(xy 57.15 162.56) (xy 72.39 162.56)
 		)
 		(stroke
@@
 	(wire
 		(pts
-			(xy 57.15 162.56) (xy 72.39 162.56)
+			(xy 77.47 121.92) (xy 77.47 138.43)
 		)
 		(stroke
@@
 	(wire
 		(pts
-			(xy 77.47 121.92) (xy 77.47 138.43)
+			(xy 138.43 142.24) (xy 144.78 142.24)
 		)
 		(stroke
@@
 	(wire
 		(pts
-			(xy 138.43 142.24) (xy 144.78 142.24)
+			(xy 77.47 105.41) (xy 77.47 121.92)
 		)
 		(stroke
@@
 	(wire
 		(pts
-			(xy 77.47 105.41) (xy 77.47 121.92)
+			(xy 57.15 146.05) (xy 72.39 146.05)
 		)
 		(stroke
@@
 			)
 		)
-		(property "Footprint" "Diode_SMD:D_SOD-123"
+		(property "Footprint" "reel:Diode_SMD"
 			(at 41.91 142.24 0)
 			(hide yes)
@@
 			)
 		)
-		(property "Footprint" "reel:SW_Hotswap_Kailh_Choc_V1_1.00u-NoClickHole"
+		(property "Footprint" "reel:SW_Hotswap_Kailh_Choc_V1V2_1.00u"
 			(at 67.31 133.35 0)
 			(hide yes)
@@
 			)
 		)
-		(property "Footprint" "Diode_SMD:D_SOD-123"
+		(property "Footprint" "reel:Diode_SMD"
 			(at 72.39 109.22 0)
 			(hide yes)
@@
 			)
 		)
-		(property "Footprint" "reel:SW_Hotswap_Kailh_Choc_V1_1.00u-NoClickHole"
+		(property "Footprint" "reel:SW_Hotswap_Kailh_Choc_V1V2_1.00u"
 			(at 82.55 100.33 0)
 			(hide yes)
@@
 			)
 		)
-		(property "Footprint" "Diode_SMD:D_SOD-123"
+		(property "Footprint" "reel:Diode_SMD"
 			(at 87.63 142.24 0)
 			(hide yes)
@@
 			)
 		)
-		(property "Footprint" "reel:SW_Hotswap_Kailh_Choc_V1_1.00u-NoClickHole"
+		(property "Footprint" "reel:SW_Hotswap_Kailh_Choc_V1V2_1.00u"
 			(at 82.55 133.35 0)
 			(hide yes)
@@
 			)
 		)
-		(property "Footprint" "reel:SW_Hotswap_Kailh_Choc_V1_1.00u-NoClickHole"
+		(property "Footprint" "reel:SW_Hotswap_Kailh_Choc_V1V2_1.00u"
 			(at 36.83 100.33 0)
 			(hide yes)
@@
 			)
 		)
-		(property "Footprint" "reel:SW_Hotswap_Kailh_Choc_V1_1.00u-NoClickHole"
+		(property "Footprint" "reel:SW_Hotswap_Kailh_Choc_V1V2_1.00u"
 			(at 52.07 133.35 0)
 			(hide yes)
@@
 			)
 		)
-		(property "Footprint" "reel:SW_Hotswap_Kailh_Choc_V1_1.00u-NoClickHole"
+		(property "Footprint" "reel:SW_Hotswap_Kailh_Choc_V1V2_1.00u"
 			(at 52.07 100.33 0)
 			(hide yes)
@@
 			)
 		)
-		(property "Footprint" "reel:SW_Hotswap_Kailh_Choc_V1_1.00u-NoClickHole"
+		(property "Footprint" "reel:SW_Hotswap_Kailh_Choc_V1V2_1.00u"
 			(at 36.83 133.35 0)
 			(hide yes)
@@
 			)
 		)
-		(property "Footprint" "reel:SW_Hotswap_Kailh_Choc_V1_1.00u-NoClickHole"
+		(property "Footprint" "reel:SW_Hotswap_Kailh_Choc_V1V2_1.00u"
 			(at 82.55 149.86 0)
 			(hide yes)
@@
 			)
 		)
-		(property "Footprint" "Diode_SMD:D_SOD-123"
+		(property "Footprint" "reel:Diode_SMD"
 			(at 72.39 142.24 0)
 			(hide yes)
@@
 			)
 		)
-		(property "Footprint" "Diode_SMD:D_SOD-123"
+		(property "Footprint" "reel:Diode_SMD"
 			(at 102.87 109.22 0)
 			(hide yes)
@@
 			)
 		)
-		(property "Footprint" "reel:SW_Hotswap_Kailh_Choc_V1_1.00u-NoClickHole"
+		(property "Footprint" "reel:SW_Hotswap_Kailh_Choc_V1V2_1.00u"
 			(at 52.07 116.84 0)
 			(hide yes)
@@
 			)
 		)
-		(property "Footprint" "Diode_SMD:D_SOD-123"
+		(property "Footprint" "reel:Diode_SMD"
 			(at 102.87 142.24 0)
 			(hide yes)
@@
 			)
 		)
-		(property "Footprint" "Diode_SMD:D_SOD-123"
+		(property "Footprint" "reel:Diode_SMD"
 			(at 57.15 125.73 0)
 			(hide yes)
@@
 			)
 		)
-		(property "Footprint" "Diode_SMD:D_SOD-123"
+		(property "Footprint" "reel:Diode_SMD"
 			(at 87.63 158.75 0)
 			(hide yes)
@@
 			)
 		)
-		(property "Footprint" "reel:SW_Hotswap_Kailh_Choc_V1_1.00u-NoClickHole"
+		(property "Footprint" "reel:SW_Hotswap_Kailh_Choc_V1V2_1.00u"
 			(at 82.55 116.84 0)
 			(hide yes)
@@
 			)
 		)
-		(property "Footprint" "Diode_SMD:D_SOD-123"
+		(property "Footprint" "reel:Diode_SMD"
 			(at 57.15 142.24 0)
 			(hide yes)
@@
 			)
 		)
-		(property "Footprint" "Diode_SMD:D_SOD-123"
+		(property "Footprint" "reel:Diode_SMD"
 			(at 87.63 125.73 0)
 			(hide yes)
@@
 			)
 		)
-		(property "Footprint" "reel:SW_Hotswap_Kailh_Choc_V1_1.00u-NoClickHole"
+		(property "Footprint" "reel:SW_Hotswap_Kailh_Choc_V1V2_1.00u"
 			(at 97.79 100.33 0)
 			(hide yes)
@@
 			)
 		)
-		(property "Footprint" "reel:SW_Hotswap_Kailh_Choc_V1_1.00u-NoClickHole"
+		(property "Footprint" "reel:SW_Hotswap_Kailh_Choc_V1V2_1.00u"
 			(at 36.83 116.84 0)
 			(hide yes)
@@
 			)
 		)
-		(property "Footprint" "reel:SW_Hotswap_Kailh_Choc_V1_1.00u-NoClickHole"
+		(property "Footprint" "reel:SW_Hotswap_Kailh_Choc_V1V2_1.00u"
 			(at 52.07 149.86 0)
 			(hide yes)
@@
 			)
 		)
-		(property "Footprint" "reel:SW_Hotswap_Kailh_Choc_V1_1.00u-NoClickHole"
+		(property "Footprint" "reel:SW_Hotswap_Kailh_Choc_V1V2_1.00u"
 			(at 97.79 133.35 0)
 			(hide yes)
@@
 			)
 		)
-		(property "Footprint" "reel:SW_Hotswap_Kailh_Choc_V1_1.00u-NoClickHole"
+		(property "Footprint" "reel:SW_Hotswap_Kailh_Choc_V1V2_1.00u"
 			(at 67.31 116.84 0)
 			(hide yes)
@@
 			)
 		)
-		(property "Footprint" "Diode_SMD:D_SOD-123"
+		(property "Footprint" "reel:Diode_SMD"
 			(at 72.39 158.75 0)
 			(hide yes)
@@
 			)
 		)
-		(property "Footprint" "reel:SW_Hotswap_Kailh_Choc_V1_1.00u-NoClickHole"
+		(property "Footprint" "reel:SW_Hotswap_Kailh_Choc_V1V2_1.00u"
 			(at 97.79 116.84 0)
 			(hide yes)
@@
 			)
 		)
-		(property "Footprint" "reel:SW_Hotswap_Kailh_Choc_V1_1.00u-NoClickHole"
+		(property "Footprint" "reel:SW_Hotswap_Kailh_Choc_V1V2_1.00u"
 			(at 67.31 149.86 0)
 			(hide yes)
@@
 			)
 		)
-		(property "Footprint" "Diode_SMD:D_SOD-123"
+		(property "Footprint" "reel:Diode_SMD"
 			(at 87.63 109.22 0)
 			(hide yes)
@@
 			)
 		)
-		(property "Footprint" "Diode_SMD:D_SOD-123"
+		(property "Footprint" "reel:Diode_SMD"
 			(at 57.15 109.22 0)
 			(hide yes)
@@
 			)
 		)
-		(property "Footprint" "Diode_SMD:D_SOD-123"
+		(property "Footprint" "reel:Diode_SMD"
 			(at 41.91 109.22 0)
 			(hide yes)
@@
 			)
 		)
-		(property "Footprint" "Diode_SMD:D_SOD-123"
+		(property "Footprint" "reel:Diode_SMD"
 			(at 41.91 125.73 0)
 			(hide yes)
@@
 			)
 		)
-		(property "Footprint" "reel:SW_Hotswap_Kailh_Choc_V1_1.00u-NoClickHole"
+		(property "Footprint" "reel:SW_Hotswap_Kailh_Choc_V1V2_1.00u"
 			(at 36.83 149.86 0)
 			(hide yes)
@@
 			)
 		)
-		(property "Footprint" "Diode_SMD:D_SOD-123"
+		(property "Footprint" "reel:Diode_SMD"
 			(at 41.91 158.75 0)
 			(hide yes)
@@
 			)
 		)
-		(property "Footprint" "Diode_SMD:D_SOD-123"
+		(property "Footprint" "reel:Diode_SMD"
 			(at 57.15 158.75 0)
 			(hide yes)
@@
 			)
 		)
-		(property "Footprint" "Diode_SMD:D_SOD-123"
+		(property "Footprint" "reel:Diode_SMD"
 			(at 72.39 125.73 0)
 			(hide yes)
@@
 			)
 		)
-		(property "Footprint" "Diode_SMD:D_SOD-123"
+		(property "Footprint" "reel:Diode_SMD"
 			(at 102.87 125.73 0)
 			(hide yes)
@@
 			)
 		)
-		(property "Footprint" "reel:SW_Hotswap_Kailh_Choc_V1_1.00u-NoClickHole"
+		(property "Footprint" "reel:SW_Hotswap_Kailh_Choc_V1V2_1.00u"
 			(at 67.31 100.33 0)
 			(hide yes)
