File: left/reel-left.kicad_sch (KiCad schematic)
At the start: 44 parts, among them J1 Conn_01x02, SW1 SW_Push, SW10 SW_Push, SW11 SW_Push, SW12 SW_Push, SW13 SW_Push, SW14 SW_Push, SW15 SW_Push, SW16 SW_Push, SW17 SW_Push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

Commit message: Update left board encoder footprint
Parts:
- SW21: footprint reel:rotary_encoder_EC05E_Vert -> reel:RotaryEncoder_BM10_3Pin
Changed lines of the file:
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@@
 			)
 		)
-		(property "Footprint" "reel:rotary_encoder_EC05E_Vert"
+		(property "Footprint" "reel:RotaryEncoder_BM10_3Pin"
 			(at 125.73 103.886 0)
 			(hide yes)
