File: left/reel-left.kicad_sch (KiCad schematic)
At the start: 44 parts, among them J1 Conn_01x02, SW1 SW_Push, SW10 SW_Push, SW11 SW_Push, SW12 SW_Push, SW13 SW_Push, SW14 SW_Push, SW15 SW_Push, SW16 SW_Push, SW17 SW_Push, SW18 SW_Push, SW19 SW_Push, SW2 SW_Push, SW20 SW_Push, SW21 RotaryEncoder, SW22 SW_SPDT, SW3 SW_Push, SW4 SW_Push, SW5 SW_Push, SW6 SW_Push, SW7 SW_Push, SW8 SW_Push, SW9 SW_Push

Commit message: Update left PCB layout
Parts:
- added D21, D22: D, Diode_SMD:D_SOD-123, symbol Device:D
- added SW21, SW22: SW_Push, reel:SideTactSwitch_2pin, symbol Switch:SW_Push
- renumbered SW22 to SW24, SW21 to SW25
Connections:
- net Col0: now also SW21.1
- net Col1: now also SW22.1
- net Row4: now reaches U1.15 (NFC1_0.09)
- net Row4: now also D21.1 (K), D22.1 (K)
- new net: D21.2 (A), SW21.2
- new net: D22.2 (A), SW22.2
- no-connect marks 8 -> 7

Commit message: Update left PCB layout
Parts:
- SW18, SW19: footprint reel:SW_Hotswap_Kailh_Choc_V1_1.00u-NoClickHole -> reel:SideTactSwitch_2pin
- SW21, SW22: footprint reel:SideTactSwitch_2pin -> reel:SW_Hotswap_Kailh_Choc_V1_1.00u-NoClickHole
Connections:
- net Col0: now also SW12.1, SW18.1; no longer SW11.1, SW16.1, SW21.1
- net Col1: now also SW13.1, SW19.1; no longer SW12.1, SW17.1, SW22.1
- net Col2: now also SW14.1, SW20.1; no longer SW13.1, SW18.1
- net Col3: now also SW15.1, SW21.1; no longer SW14.1, SW19.1
- net Col4: now also SW16.1, SW22.1; no longer SW15.1, SW20.1
- net Row1: now also D11.1 (K)
- net Row2: now also D16.1 (K), D17.1 (K); no longer D11.1 (K)
- net Row3: now also D21.1 (K), D22.1 (K); no longer D16.1 (K), D17.1 (K)
- removed net Row4: D21.1 (K), D22.1 (K), U1.15 (NFC1_0.09)
- new net Col5: SW11.1, SW17.1, U1.15 (NFC1_0.09)
Other:
- moved on the sheet: D11, D12, D13, D14, D15, D16, D17, D18, D19, D20, D21, D22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

Commit message: Update ReeL KiCad libraries and board
Parts:
- U1: symbol roba:XIAO-nRF52840 -> reel:XIAO-nRF52840
Changed lines of the file:
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@@
 	)
 	(symbol
-		(lib_id "roba:XIAO-nRF52840")
+		(lib_id "reel:XIAO-nRF52840")
 		(at 27.94 25.4 0)
 		(unit 1)

Commit message: Update ReeL KiCad board files
Parts:
- D1, D10, D11, D12, D13, D14, D15, D16, D17, D18, D19, D2, D20, D21, D22, D3, D4, D5, D6, D7, D8, D9: footprint Diode_SMD:D_SOD-123 -> reel:Diode_SMD
- SW1, SW10, SW11, SW12, SW13, SW14, SW15, SW16, SW17, SW2, SW20, SW21, SW22, SW3, SW4, SW5, SW6, SW7, SW8, SW9: footprint reel:SW_Hotswap_Kailh_Choc_V1_1.00u-NoClickHole -> reel:SW_Hotswap_Kailh_Choc_V1V2_1.00u
Connections:
- net RotA: now also U1.10 (P1.14_D9_MISO); no longer U1.11 (P1.15_D10_MOSI)
- net RotB: now also U1.11 (P1.15_D10_MOSI); no longer U1.10 (P1.14_D9_MISO)

Commit message: Update ReeL switch footprints and board layouts
Parts:
- SW18: footprint reel:SideTactSwitch_2pin -> reel:Switch_E-Switch_TS2_Vertical_THT
- SW19: footprint reel:SideTactSwitch_2pin -> reel:Switch_E-Switch_TS2_Vertical_THT_Mirrored
Changed lines of the file:
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@@
 			)
 		)
-		(property "Footprint" "reel:SideTactSwitch_2pin"
+		(property "Footprint" "reel:Switch_E-Switch_TS2_Vertical_THT"
 			(at 36.83 149.86 0)
 			(hide yes)
@@
 			)
 		)
-		(property "Footprint" "reel:SideTactSwitch_2pin"
+		(property "Footprint" "reel:Switch_E-Switch_TS2_Vertical_THT_Mirrored"
 			(at 52.07 149.86 0)
 			(hide yes)
