File: hardware/pcb/right-top/reel-right-top.kicad_sch (KiCad schematic)
At the start: 42 parts, among them J1 Conn_01x02, SW1 SW_Push, SW10 SW_Push, SW11 SW_Push, SW12 SW_Push, SW13 SW_Push, SW14 SW_Push, SW15 SW_Push, SW16 SW_Push, SW17 SW_Push, SW18 SW_Push, SW19 SW_Push, SW2 SW_Push, SW22 SW_SPDT, SW3 SW_Push, SW4 SW_Push, SW5 SW_Push, SW6 SW_Push, SW7 SW_Push, SW8 SW_Push, SW9 SW_Push

Commit message: Update ReeL hardware and fabrication assets
Parts:
- added J3: Conn_01x05, reel:Display_BeeKeeb_MIP_1.08in_LS011B7DH03, symbol Connector_Generic:Conn_01x05
Connections:
- net 3.3V: now also J3.2 (Pin_2)
- net GND: now also J3.1 (Pin_1)
- net SI: now reaches U1.17 (NFC3_0.16)
- net SI: now also J3.3 (Pin_3)
- net SCK: now reaches U1.18 (NFC4_1.00)
- net SCK: now also J3.4 (Pin_4)
- net CS: now reaches U1.19 (NFC5_1.10)
- net CS: now also J3.5 (Pin_5)
- no-connect marks 6 -> 3
