File: hardware/pcb/left/reel-left.kicad_pcb (KiCad board)
At the start: 2 copper layers, 150.6 x 100.3 mm, 54 parts, among them J1 Conn_01x02, J2 Conn_01x05, SW1 SW_Push, SW10 SW_Push, SW11 SW_Push, SW12 SW_Push, SW13 SW_Push, SW14 SW_Push, SW15 SW_Push, SW16 SW_Push, SW17 SW_Push, SW18 SW_Push, SW19 SW_Push, SW2 SW_Push, SW20 SW_Push, SW21 SW_Push, SW22 SW_Push, SW24 SW_SPDT, SW25 RotaryEncoder, SW3 SW_Push, SW4 SW_Push, SW5 SW_Push, SW6 SW_Push, SW7 SW_Push, SW8 SW_Push, SW9 SW_Push

Commit message: Add LCD status firmware and update project assets
Routing:
- net SCK: track 38.0 -> 33.3 mm, vias 1 -> 0
- net Col5: track 174.6 -> 171.2 mm
Changed lines of the file:
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@@
+	)
+	(segment
+		(start 202.75 79.25)
+		(end 202.75 83)
+		(width 0.25)
+		(layer "F.Cu")
+		(net "Col5")
+	)
+	(segment
+		(start 145.1084 114.25)
+		(end 138.8584 108)
+		(width 0.25)
+		(layer "F.Cu")
+		(net "Col5")
+	)
+	(segment
+		(start 194.75 112.25)
+		(end 193.75 113.25)
+		(width 0.25)
+		(layer "F.Cu")
+		(net "Col5")
+	)
+	(segment
+		(start 199.75 86)
+		(end 199.75 105.770786)
+		(width 0.25)
+		(layer "F.Cu")
+		(net "Col5")
+	)
+	(segment
+		(start 138.8584 108)
+		(end 106 108)
+		(width 0.25)
+		(layer "F.Cu")
+		(net "Col5")
+	)
+	(segment
+		(start 202.077318 78.577318)
+		(end 202.75 79.25)
+		(width 0.25)
+		(layer "F.Cu")
+		(net "Col5")
+	)
+	(segment
+		(start 202.75 83)
+		(end 199.75 86)
+		(width 0.25)
+		(layer "F.Cu")
+		(net "Col5")
 	)
 	(segment
 		(start 164.25 115)
+		(end 163.5 114.25)
+		(width 0.25)
+		(layer "F.Cu")
+		(net "Col5")
+	)
+	(segment
+		(start 106 108)
+		(end 104.5 106.5)
+		(width 0.25)
+		(layer "F.Cu")
+		(net "Col5")
+	)
+	(segment
+		(start 187.636396 115)
+		(end 164.25 115)
+		(width 0.25)
+		(layer "F.Cu")
+		(net "Col5")
+	)
+	(segment
+		(start 163.5 114.25)
+		(end 145.1084 114.25)
+		(width 0.25)
+		(layer "F.Cu")
+		(net "Col5")
+	)
+	(segment
+		(start 193.75 113.25)
+		(end 189.386396 113.25)
+		(width 0.25)
+		(layer "F.Cu")
+		(net "Col5")
+	)
+	(segment
+		(start 199.75 105.770786)
+		(end 194.75 110.770786)
+		(width 0.25)
+		(layer "F.Cu")
+		(net "Col5")
+	)
+	(segment
+		(start 189.386396 113.25)
 		(end 187.636396 115)
 		(width 0.25)
@@
 	)
 	(segment
-		(start 187.636396 115)
-		(end 189.386396 113.25)
-		(width 0.25)
-		(layer "F.Cu")
-		(net "Col5")
-	)
-	(segment
-		(start 189.386396 113.25)
-		(end 198.75 113.25)
-		(width 0.25)
-		(layer "F.Cu")
-		(net "Col5")
-	)
-	(segment
-		(start 199.25 107)
-		(end 199.25 105.5)
-		(width 0.25)
-		(layer "F.Cu")
-		(net "Col5")
-	)
-	(segment
-		(start 199.75 107.5)
-		(end 199.25 107)
-		(width 0.25)
-		(layer "F.Cu")
-		(net "Col5")
-	)
-	(segment
-		(start 106 108)
-		(end 138.8584 108)
-		(width 0.25)
-		(layer "F.Cu")
-		(net "Col5")
-	)
-	(segment
-		(start 199.75 86)
-		(end 202.75 83)
-		(width 0.25)
-		(layer "F.Cu")
-		(net "Col5")
-	)
-	(segment
-		(start 145.1084 114.25)
-		(end 163.5 114.25)
-		(width 0.25)
-		(layer "F.Cu")
-		(net "Col5")
-	)
-	(segment
-		(start 198.75 113.25)
-		(end 199.75 112.25)
-		(width 0.25)
-		(layer "F.Cu")
-		(net "Col5")
-	)
-	(segment
-		(start 87 106.5)
-		(end 104.5 106.5)
-		(width 0.25)
-		(layer "F.Cu")
-		(net "Col5")
-	)
-	(segment
-		(start 199.75 112.25)
-		(end 199.75 107.5)
+		(start 202.077318 76.037693)
+		(end 202.077318 78.577318)
+		(width 0.25)
+		(layer "F.Cu")
+		(net "Col5")
+	)
+	(segment
+		(start 194.75 110.770786)
+		(end 194.75 112.25)
 		(width 0.25)
 		(layer "F.Cu")
@@
 	(segment
 		(start 104.5 106.5)
-		(end 106 108)
-		(width 0.25)
-		(layer "F.Cu")
-		(net "Col5")
-	)
-	(segment
-		(start 138.8584 108)
-		(end 145.1084 114.25)
-		(width 0.25)
-		(layer "F.Cu")
-		(net "Col5")
-	)
-	(segment
-		(start 202.077318 78.577318)
-		(end 202.077318 76.037693)
-		(width 0.25)
-		(layer "F.Cu")
-		(net "Col5")
-	)
-	(segment
-		(start 199.25 105.5)
-		(end 199.75 105)
-		(width 0.25)
-		(layer "F.Cu")
-		(net "Col5")
-	)
-	(segment
-		(start 202.75 83)
-		(end 202.75 79.25)
-		(width 0.25)
-		(layer "F.Cu")
-		(net "Col5")
-	)
-	(segment
-		(start 199.75 105)
-		(end 199.75 86)
-		(width 0.25)
-		(layer "F.Cu")
-		(net "Col5")
-	)
-	(segment
-		(start 202.75 79.25)
-		(end 202.077318 78.577318)
-		(width 0.25)
-		(layer "F.Cu")
-		(net "Col5")
-	)
-	(segment
-		(start 163.5 114.25)
-		(end 164.25 115)
+		(end 87 106.5)
 		(width 0.25)
 		(layer "F.Cu")
@@
 	)
 	(segment
+		(start 201 105.935)
+		(end 201 105.25)
+		(width 0.25)
+		(layer "F.Cu")
+		(net "SCK")
+	)
+	(segment
 		(start 201 86)
 		(end 204 83)
@@
 	)
 	(segment
+		(start 195.935 111)
+		(end 201 105.935)
+		(width 0.25)
+		(layer "F.Cu")
+		(net "SCK")
+	)
+	(segment
 		(start 204 83)
 		(end 204 81)
@@
 		(net "SCK")
 	)
-	(segment
-		(start 200 106.25)
-		(end 201 105.25)
-		(width 0.25)
-		(layer "F.Cu")
-		(net "SCK")
-	)
-	(via
-		(at 200 106.25)
-		(size 0.6)
-		(drill 0.3)
-		(layers "F.Cu" "B.Cu")
-		(net "SCK")
-	)
-	(segment
-		(start 195.935 111.935)
-		(end 196.5 112.5)
-		(width 0.25)
-		(layer "B.Cu")
-		(net "SCK")
-	)
-	(segment
-		(start 195.935 111)
-		(end 195.935 111.935)
-		(width 0.25)
-		(layer "B.Cu")
-		(net "SCK")
-	)
-	(segment
-		(start 196.5 112.5)
-		(end 199.25 112.5)
-		(width 0.25)
-		(layer "B.Cu")
-		(net "SCK")
-	)
-	(segment
-		(start 199.25 112.5)
-		(end 199.75 112)
-		(width 0.25)
-		(layer "B.Cu")
-		(net "SCK")
-	)
-	(segment
-		(start 199.75 112)
-		(end 199.75 106.5)
-		(width 0.25)
-		(layer "B.Cu")
-		(net "SCK")
-	)
-	(segment
-		(start 200 106.25)
-		(end 199.75 106.5)
-		(width 0.25)
-		(layer "B.Cu")
-		(net "SCK")
-	)
